Commit message: Add colors and remove duplicates

File: src/my_robot/urdf/my_robot.xacro (robot description, xacro)
@@ -1,178 +1,196 @@
 <?xml version='1.0'?>
 <robot name="my_robot" xmlns:xacro="http://www.ros.org/wiki/xacro">
-                                                  <link name="robot_footprint"></link>
-                                                  <joint name="robot_footprint_joint" type="fixed">
-                                                    <origin xyz="0 0 0" rpy="0 0 0" />
-                                                    <parent link="robot_footprint"/>
-                                                    <child link="chassis" />
-                                                  </joint>
-                                                  <link name='chassis'>
-                                                    <pose>0 0 0.05 0 0 0</pose>
-                                                    <inertial>
-                                                      <mass value="15.0"/>
-                                                      <origin xyz="0.0 0 0" rpy=" 0 0 0"/>
-                                                      <inertia
-                                                          ixx="0.1" ixy="0" ixz="0"
-                                                          iyy="0.1" iyz="0"
-                                                          izz="0.1"
-                                                      />
-                                                    </inertial>
-                                                    <collision name='collision'>
-                                                      <origin xyz="0 0 0" rpy=" 0 0 0"/>
-                                                      <geometry>
-                                                        <cylinder radius="0.2" length="0.05"/>
-                                                      </geometry>
-                                                    </collision>
-                                                    <visual name='chassis_visual'>
-                                                      <origin xyz="0 0 0" rpy=" 0 0 0"/>
-                                                      <geometry>
-                                                        <cylinder radius="0.2" length="0.05"/>
-                                                      </geometry>
-                                                    </visual>
-                                                    <collision name='back_caster_collision'>
-                                                      <origin xyz="-0.15 0 -0.02" rpy=" 0 0 0"/>
-                                                      <geometry>
-                                                        <sphere radius="0.0199"/>
-                                                      </geometry>
-                                                    </collision>
-                                                    <visual name='back_caster_visual'>
-                                                      <origin xyz="-0.15 0 -0.02" rpy=" 0 0 0"/>
-                                                      <geometry>
-                                                        <sphere radius="0.02"/>
-                                                      </geometry>
-                                                    </visual>
-                                                    <collision name='front_caster_collision'>
-                                                      <origin xyz="0.15 0 -0.02" rpy=" 0 0 0"/>
-                                                      <geometry>
-                                                        <sphere radius="0.0199"/>
-                                                      </geometry>
-                                                    </collision>
-                                                    <visual name='front_caster_visual'>
-                                                      <origin xyz="0.15 0 -0.02" rpy=" 0 0 0"/>
-                                                      <geometry>
-                                                        <sphere radius="0.02"/>
-                                                      </geometry>
-                                                    </visual>
-                                                  </link>
-                                                  <link name="left_wheel">
-                                                    <collision name='collision'>
-                                                      <origin xyz="0 0 0" rpy=" 0 1.57 1.57"/>
-                                                      <geometry>
-                                                        <cylinder radius="0.03" length="0.02"/>
-                                                      </geometry>
-                                                    </collision>
-                                                    <visual name='visual'>
-                                                      <origin xyz="0 0 0" rpy=" 0 1.57 1.57"/>
-                                                      <geometry>
-                                                        <cylinder radius="0.03" length="0.02"/>
-                                                      </geometry>
-                                                    </visual>
-                                                    <inertial>
-                                                      <mass value="5.0"/>
-                                                      <origin xyz="0.0 0 0" rpy=" 0 0 0"/>
-                                                      <inertia
-                                                          ixx="0.1" ixy="0" ixz="0"
-                                                          iyy="0.1" iyz="0"
-                                                          izz="0.1"
-                                                      />
-                                                    </inertial>
-                                                  </link>
-                                                  <link name="right_wheel">
-                                                    <collision name='collision'>
-                                                      <origin xyz="0 0 0" rpy=" 0 1.57 1.57"/>
-                                                      <geometry>
-                                                        <cylinder radius="0.03" length="0.02"/>
-                                                      </geometry>
-                                                    </collision>
-                                                    <visual name='visual'>
-                                                      <origin xyz="0 0 0" rpy=" 0 1.57 1.57"/>
-                                                      <geometry>
-                                                        <cylinder radius="0.03" length="0.02"/>
-                                                      </geometry>
-                                                    </visual>
-                                                    <inertial>
-                                                      <mass value="5.0"/>
-                                                      <origin xyz="0.0 0 0" rpy=" 0 0 0"/>
-                                                      <inertia
-                                                          ixx="0.1" ixy="0" ixz="0"
-                                                          iyy="0.1" iyz="0"
-                                                          izz="0.1"
-                                                      />
-                                                    </inertial>
-                                                  </link>
-                                                  <joint name="left_wheel_hinge" type="continuous">
-                                                    <origin xyz="0 0.15 -0.01" rpy="0 0 0" />
-                                                    <parent link="chassis"/>
-                                                    <child link="left_wheel" />
-                                                    <axis xyz="0 1 0" rpy="0 0 0"/>
-                                                    <limit effort="1000" velocity="1000"/>
-                                                    <dynamic damping="1.0" friction="1.0"/>
-                                                  </joint>
-                                                  <joint name="right_wheel_hinge" type="continuous">
-                                                    <origin xyz="0 -0.15 -0.01" rpy="0 0 0" />
-                                                    <parent link="chassis"/>
-                                                    <child link="right_wheel" />
-                                                    <axis xyz="0 1 0" rpy="0 0 0"/>
-                                                    <limit effort="1000" velocity="1000"/>
-                                                    <dynamic damping="1.0" friction="1.0"/>
-                                                  </joint>
-                                                  <link name="camera">
-                                                    <inertial>
-                                                      <mass value="0.1"/>
-                                                      <origin xyz="0.0 0 0" rpy=" 0 0 0"/>
-                                                      <inertia
-                                                          ixx="1e-6" ixy="0" ixz="0"
-                                                          iyy="1e-6" iyz="0"
-                                                          izz="1e-6"
-                                                      />
-                                                    </inertial>
-                                                    <collision name='collision'>
-                                                      <origin xyz="0 0 0" rpy=" 0 0 0"/>
-                                                      <geometry>
-                                                        <box size="0.05 0.05 0.05"/>
-                                                      </geometry>
-                                                    </collision>
-                                                    <visual name='visual'>
-                                                      <origin xyz="0 0 0" rpy=" 0 0 0"/>
-                                                      <geometry>
-                                                        <box size="0.05 0.05 0.05"/>
-                                                      </geometry>
-                                                    </visual>
-                                                  </link>
-                                                  <joint name="camera_joint" type="fixed">
-                                                    <origin xyz="0.2 0 0" rpy="0 0 0" />
-                                                    <parent link="chassis"/>
-                                                    <child link="camera" />
-                                                    <axis xyz="0 1 0" rpy="0 0 0"/>
-                                                  </joint>
-                                                  <link name="hokuyo">
-                                                  <inertial>
-                                                    <mass value="1e-5"/>
-                                                    <origin xyz="0.0 0 0" rpy=" 0 0 0"/>
-                                                    <inertia
-                                                        ixx="1e-6" ixy="0" ixz="0"
-                                                        iyy="1e-6" iyz="0"
-                                                        izz="1e-6"
-                                                    />
-                                                  </inertial>
-                                                  <collision name='collision'>
-                                                    <origin xyz="0 0 0" rpy=" 0 0 0"/>
-                                                    <geometry>
-                                                      <box size="0.1 0.1 0.1"/>
-                                                    </geometry>
-                                                  </collision>
-                                                  <visual name='visual'>
-                                                    <origin xyz="0 0 0" rpy=" 0 0 0"/>
-                                                    <geometry>
-                                                      <mesh filename="package://my_robot/meshes/hokuyo.dae"/>
-                                                    </geometry>
-                                                  </visual>
-                                                  </link>
-                                                  <joint name="hokuyo_joint" type="fixed">
-                                                    <origin xyz="0.17 0 0.05" rpy="0 0 0" />
-                                                    <parent link="chassis"/>
-                                                    <child link="hokuyo" />
-                                                    <axis xyz="0 1 0" rpy="0 0 0"/>
-                                                  </joint>
-                                                  <xacro:include filename="$(find my_robot)/urdf/my_robot.gazebo" />
+      <xacro:include filename="$(find my_robot)/urdf/my_robot.gazebo" />
+      <link name="robot_footprint"></link>
+      <joint name="robot_footprint_joint" type="fixed">
+        <origin xyz="0 0 0" rpy="0 0 0" />
+        <parent link="robot_footprint"/>
+        <child link="chassis" />
+      </joint>
+      <link name='chassis'>
+        <pose>0 0 0.05 0 0 0</pose>
+        <inertial>
+          <mass value="15.0"/>
+          <origin xyz="0.0 0 0" rpy=" 0 0 0"/>
+          <inertia
+              ixx="0.1" ixy="0" ixz="0"
+              iyy="0.1" iyz="0"
+              izz="0.1"
+          />
+        </inertial>
+        <collision name='collision_chassis'>
+          <origin xyz="0 0 0" rpy=" 0 0 0"/>
+          <geometry>
+            <cylinder radius="0.2" length="0.05"/>
+          </geometry>
+        </collision>
+        <visual name='chassis_visual'>
+          <origin xyz="0 0 0" rpy=" 0 0 0"/>
+          <geometry>
+            <cylinder radius="0.2" length="0.05"/>
+          </geometry>
+          <material name="chassis_material">
+            <color rgba="0 0 1 1"/>
+          </material>
+        </visual>
+        <collision name='back_caster_collision'>
+          <origin xyz="-0.15 0 -0.02" rpy=" 0 0 0"/>
+          <geometry>
+            <sphere radius="0.0199"/>
+          </geometry>
+        </collision>
+        <visual name='back_caster_visual'>
+          <origin xyz="-0.15 0 -0.02" rpy=" 0 0 0"/>
+          <geometry>
+            <sphere radius="0.02"/>
+          </geometry>
+          <material name="back_caster_material">
+            <color rgba="0 0 0 1"/>
+          </material>
+        </visual>
+        <collision name='front_caster_collision'>
+          <origin xyz="0.15 0 -0.02" rpy=" 0 0 0"/>
+          <geometry>
+            <sphere radius="0.0199"/>
+          </geometry>
+        </collision>
+        <visual name='front_caster_visual'>
+          <origin xyz="0.15 0 -0.02" rpy=" 0 0 0"/>
+          <geometry>
+            <sphere radius="0.02"/>
+          </geometry>
+          <material name="front_caster_material">
+            <color rgba="0 0 0 1"/>
+          </material>
+        </visual>
+      </link>
+      <link name="left_wheel">
+        <collision name='left_wheel_collision'>
+          <origin xyz="0 0 0" rpy=" 0 1.57 1.57"/>
+          <geometry>
+            <cylinder radius="0.03" length="0.02"/>
+          </geometry>
+        </collision>
+        <visual name='left_wheel_visual'>
+          <origin xyz="0 0 0" rpy=" 0 1.57 1.57"/>
+          <geometry>
+            <cylinder radius="0.03" length="0.02"/>
+          </geometry>
+          <material name="left_wheel_material">
+            <color rgba="0 0 0 1"/>
+          </material>
+        </visual>
+        <inertial>
+          <mass value="5.0"/>
+          <origin xyz="0.0 0 0" rpy=" 0 0 0"/>
+          <inertia
+              ixx="0.1" ixy="0" ixz="0"
+              iyy="0.1" iyz="0"
+              izz="0.1"
+          />
+        </inertial>
+      </link>
+      <link name="right_wheel">
+        <collision name='right_wheel_collision'>
+          <origin xyz="0 0 0" rpy=" 0 1.57 1.57"/>
+          <geometry>
+            <cylinder radius="0.03" length="0.02"/>
+          </geometry>
+        </collision>
+        <visual name='right_wheel_visual'>
+          <origin xyz="0 0 0" rpy=" 0 1.57 1.57"/>
+          <geometry>
+            <cylinder radius="0.03" length="0.02"/>
+          </geometry>
+          <material name="right_wheel_material">
+            <color rgba="0 0 0 1"/>
+          </material>
+        </visual>
+        <inertial>
+          <mass value="5.0"/>
+          <origin xyz="0.0 0 0" rpy=" 0 0 0"/>
+          <inertia
+              ixx="0.1" ixy="0" ixz="0"
+              iyy="0.1" iyz="0"
+              izz="0.1"
+          />
+        </inertial>
+      </link>
+      <joint name="left_wheel_hinge" type="continuous">
+        <origin xyz="0 0.15 -0.01" rpy="0 0 0" />
+        <parent link="chassis"/>
+        <child link="left_wheel" />
+        <axis xyz="0 1 0" rpy="0 0 0"/>
+        <limit effort="1000" velocity="1000"/>
+        <dynamic damping="1.0" friction="1.0"/>
+      </joint>
+      <joint name="right_wheel_hinge" type="continuous">
+        <origin xyz="0 -0.15 -0.01" rpy="0 0 0" />
+        <parent link="chassis"/>
+        <child link="right_wheel" />
+        <axis xyz="0 1 0" rpy="0 0 0"/>
+        <limit effort="1000" velocity="1000"/>
+        <dynamic damping="1.0" friction="1.0"/>
+      </joint>
+      <link name="camera">
+        <inertial>
+          <mass value="0.1"/>
+          <origin xyz="0.0 0 0" rpy=" 0 0 0"/>
+          <inertia
+              ixx="1e-6" ixy="0" ixz="0"
+              iyy="1e-6" iyz="0"
+              izz="1e-6"
+          />
+        </inertial>
+        <collision name='collision_camera'>
+          <origin xyz="0 0 0" rpy=" 0 0 0"/>
+          <geometry>
+            <box size="0.05 0.05 0.05"/>
+          </geometry>
+        </collision>
+        <visual name='camera_visual'>
+          <origin xyz="0 0 0" rpy=" 0 0 0"/>
+          <geometry>
+            <box size="0.05 0.05 0.05"/>
+          </geometry>
+          <material name="camera_material">
+            <color rgba="0 1 0 1"/>
+          </material>
+        </visual>
+      </link>
+      <joint name="camera_joint" type="fixed">
+        <origin xyz="0.225 0 0" rpy="0 0 0" />
+        <parent link="chassis"/>
+        <child link="camera" />
+        <axis xyz="0 1 0" rpy="0 0 0"/>
+      </joint>
+      <link name="hokuyo">
+      <inertial>
+        <mass value="1e-5"/>
+        <origin xyz="0.0 0 0" rpy=" 0 0 0"/>
+        <inertia
+            ixx="1e-6" ixy="0" ixz="0"
+            iyy="1e-6" iyz="0"
+            izz="1e-6"
+        />
+      </inertial>
+      <collision name='collision_hokuyo'>
+        <origin xyz="0 0 0" rpy=" 0 0 0"/>
+        <geometry>
+          <box size="0.1 0.1 0.1"/>
+        </geometry>
+      </collision>
+      <visual name='visual_hokuyo'>
+        <origin xyz="0 0 0" rpy=" 0 0 0"/>
+        <geometry>
+          <mesh filename="package://my_robot/meshes/hokuyo.dae"/>
+        </geometry>
+      </visual>
+      </link>
+      <joint name="hokuyo_joint" type="fixed">
+        <origin xyz="0.17 0 0.05" rpy="0 0 0" />
+        <parent link="chassis"/>
+        <child link="hokuyo" />
+        <axis xyz="0 1 0" rpy="0 0 0"/>
+      </joint>
 </robot>
